File: Splitter/RP-HAT-Splitter/RP-HAT-Splitter.kicad_sch (KiCad schematic)
At the start: 16 parts, among them J1 GPIO, J2 Conn_01x04_Socket, J3 Conn_01x04_Socket, J4 Conn_01x04_Socket, J5 Conn_01x04_Socket, J6 Conn_01x04_Socket, J7 Conn_01x04_Socket, U1 CAT24C256

Commit message: asd
Parts:
- added J102: I2C1-Multi0, Connector_JST:JST_SH_SM04B-SRSS-TB_1x04-1MP_P1.00mm_Horizontal, symbol Connector:Conn_01x04_Socket
- added J103: I2C1-Multi7, Connector_JST:JST_SH_SM04B-SRSS-TB_1x04-1MP_P1.00mm_Horizontal, symbol Connector:Conn_01x04_Socket
- added J105: I2C1-Multi1, Connector_JST:JST_SH_SM04B-SRSS-TB_1x04-1MP_P1.00mm_Horizontal, symbol Connector:Conn_01x04_Socket
- added J106: I2C1-Multi6, Connector_JST:JST_SH_SM04B-SRSS-TB_1x04-1MP_P1.00mm_Horizontal, symbol Connector:Conn_01x04_Socket
- added J108: I2C1-Multi2, Connector_JST:JST_SH_SM04B-SRSS-TB_1x04-1MP_P1.00mm_Horizontal, symbol Connector:Conn_01x04_Socket
- added J109: I2C1-Multi5, Connector_JST:JST_SH_SM04B-SRSS-TB_1x04-1MP_P1.00mm_Horizontal, symbol Connector:Conn_01x04_Socket
- added J111: I2C1-Multi3, Connector_JST:JST_SH_SM04B-SRSS-TB_1x04-1MP_P1.00mm_Horizontal, symbol Connector:Conn_01x04_Socket
- added J112: I2C1-Multi4, Connector_JST:JST_SH_SM04B-SRSS-TB_1x04-1MP_P1.00mm_Horizontal, symbol Connector:Conn_01x04_Socket
- added R103, R104, R105, R106, R107, R108, R109, R110, R111, R112, R113, R114, R115, R116, R117, R118, R119: 4k7, Resistor_SMD:R_1206_3216Metric_Pad1.30x1.75mm_HandSolder, symbol Device:R
- added U102: PCA9548ARGE, Package_DFN_QFN:Texas_RGE0024C_EP2.1x2.1mm, symbol Interface_Expansion:PCA9548ARGE
- J104: renamed from J2; value Conn_01x04_Socket -> I2C1-Normal
- J107: renamed from J3; value Conn_01x04_Socket -> I2C1-Normal
- J110: renamed from J4; value Conn_01x04_Socket -> I2C1-Normal
- J113: renamed from J5; value Conn_01x04_Socket -> I2C1-Normal
- J114: renamed from J6; value Conn_01x04_Socket -> I2C1-Normal
- J115: renamed from J7; value Conn_01x04_Socket -> I2C1-Normal
- renumbered C1 to C101, H4 to H101, H3 to H102, H2 to H103, H1 to H104, J1 to J101, JP1 to JP101, R1 to R101, R2 to R102, U1 to U101
Connections:
- net +3V3: now also J102.1 (Pin_1), J103.1 (Pin_1), J105.1 (Pin_1), J106.1 (Pin_1), J108.1 (Pin_1), J109.1 (Pin_1), J111.1 (Pin_1), J112.1 (Pin_1), R103.2, R104.2, R105.2, R106.2, R107.2, R108.2, R109.2, R110.2, R111.2, R112.2, R113.2, R114.2, R115.2, R116.2, R117.2, R118.2, R119.2, U102.21 (VCC)
- net GND: now also J102.2 (Pin_2), J103.2 (Pin_2), J105.2 (Pin_2), J106.2 (Pin_2), J108.2 (Pin_2), J109.2 (Pin_2), J111.2 (Pin_2), J112.2 (Pin_2), U102.18 (A2), U102.22 (A0), U102.23 (A1), U102.9 (GND)
- net I2C1_SCL: now also U102.19 (SCL)
- net I2C1_SDA: now also U102.20 (SDA)
- new net: J106.4 (Pin_4), R115.1, U102.15 (SC6)
- new net: J103.3 (Pin_3), R118.1, U102.16 (SD7)
- new net: J102.3 (Pin_3), R104.1, U102.1 (SD0)
- new net: J102.4 (Pin_4), R103.1, U102.2 (SC0)
- new net: J111.3 (Pin_3), R110.1, U102.7 (SD3)
- new net: J109.3 (Pin_3), R114.1, U102.12 (SD5)
- new net: R119.1, U102.24 (~{RESET})
- new net: J112.3 (Pin_3), R112.1, U102.10 (SD4)
- new net: J112.4 (Pin_4), R111.1, U102.11 (SC4)
- new net: J109.4 (Pin_4), R113.1, U102.13 (SC5)
- new net: J106.3 (Pin_3), R116.1, U102.14 (SD6)
- new net: J103.4 (Pin_4), R117.1, U102.17 (SC7)
- new net: J105.3 (Pin_3), R106.1, U102.3 (SD1)
- new net: J105.4 (Pin_4), R105.1, U102.4 (SC1)
- new net: J108.3 (Pin_3), R108.1, U102.5 (SD2)
- new net: J108.4 (Pin_4), R107.1, U102.6 (SC2)
- new net: J111.4 (Pin_4), R109.1, U102.8 (SC3)
